Commit message: add xarm6 with puhser.

File: xarm/xarm6_with_gripper.urdf (robot description, URDF)
Before this commit: robot xarm6_with_gripper, 15 links, 14 joints
Links:
- removed link left_finger
- removed link left_inner_knuckle
- removed link left_outer_knuckle
- removed link right_finger
- removed link right_inner_knuckle
- removed link right_outer_knuckle
- link link1: geometry collision mesh filename=xarm_description/meshes/xarm6/collision/link1_vhacd.obj; visual mesh filename=xarm_description/meshes/xarm6/visual/link1.obj
- link link2: geometry collision mesh filename=xarm_description/meshes/xarm6/collision/link2_vhacd2.obj; visual mesh filename=xarm_description/meshes/xarm6/visual/link2.obj
- link link3: geometry collision mesh filename=xarm_description/meshes/xarm6/collision/link3_vhacd.obj; visual mesh filename=xarm_description/meshes/xarm6/visual/link3.obj
- link link4: geometry collision mesh filename=xarm_description/meshes/xarm6/collision/link4_vhacd.obj; visual mesh filename=xarm_description/meshes/xarm6/visual/link4.obj
- link link5: geometry collision mesh filename=xarm_description/meshes/xarm6/collision/link5_vhacd.obj; visual mesh filename=xarm_description/meshes/xarm6/visual/link5.obj
- link link6: geometry collision mesh filename=xarm_description/meshes/xarm6/visual/link6.obj; visual mesh filename=xarm_description/meshes/xarm6/visual/link6.obj
- link link_base: geometry collision mesh filename=xarm_description/meshes/xarm6/collision/base_vhacd.obj; visual mesh filename=xarm_description/meshes/xarm6/visual/base.obj
- link xarm_gripper_base_link: geometry collision mesh filename=xarm_gripper/meshes/finger_v2.obj; visual mesh filename=xarm_gripper/meshes/finger_v2.obj
Joints:
- removed joint drive_joint
- removed joint left_finger_joint
- removed joint left_inner_knuckle_joint
- removed joint right_finger_joint
- removed joint right_inner_knuckle_joint
- removed joint right_outer_knuckle_joint

File: xarm/xarm6_with_gripper_2.urdf (robot description, URDF)
Before this commit: robot xarm6, 8 links, 7 joints
Links:
- added link left_finger, mass 0.048304; collision mesh filename=xarm_gripper/meshes/finger.obj; visual mesh filename=xarm_gripper/meshes/finger.obj
- added link left_inner_knuckle, mass 0.0230125781256706; collision mesh filename=xarm_gripper/meshes/left_inner_knuckle.obj; visual mesh filename=xarm_gripper/meshes/left_inner_knuckle.obj
- added link left_outer_knuckle, mass 0.033618; collision mesh filename=xarm_gripper/meshes/left_outer_knuckle.obj; visual mesh filename=xarm_gripper/meshes/left_outer_knuckle.obj
- added link right_finger, mass 0.048304; collision mesh filename=xarm_gripper/meshes/finger.obj; visual mesh filename=xarm_gripper/meshes/finger.obj
- added link right_inner_knuckle, mass 0.023013; collision mesh filename=xarm_gripper/meshes/right_inner_knuckle.obj; visual mesh filename=xarm_gripper/meshes/right_inner_knuckle.obj
- added link right_outer_knuckle, mass 0.033618; collision mesh filename=xarm_gripper/meshes/right_outer_knuckle.obj; visual mesh filename=xarm_gripper/meshes/right_outer_knuckle.obj
- added link xarm_gripper_base_link, mass 0.54156; collision mesh filename=xarm_gripper/meshes/finger.obj; visual mesh filename=xarm_gripper/meshes/finger.obj
- link link2: geometry collision mesh filename=xarm_description/meshes/xarm6/collision/link2_vhacd2.obj; visual mesh filename=xarm_description/meshes/xarm6/visual/link2.obj
- link link6: geometry collision mesh filename=xarm_description/meshes/xarm6/visual/link6.obj; visual mesh filename=xarm_description/meshes/xarm6/visual/link6.obj
Joints:
- added joint drive_joint: type revolute, parent xarm_gripper_base_link, child left_outer_knuckle, origin xyz=0 0.035 0.059098 rpy=0 0 0, axis 1 0 0, limit lower=0 upper=0.85 effort=50 velocity=2
- added joint gripper_fix: type fixed, parent link6, child xarm_gripper_base_link, origin xyz=0 0 0 rpy=0 0 0
- added joint left_finger_joint: type revolute, parent left_outer_knuckle, child left_finger, origin xyz=0 0.035465 0.042039 rpy=0 0 0, axis -1 0 0, limit lower=0 upper=0.85 effort=50 velocity=2, mimic joint=drive_joint multiplier=1 offset=0
- added joint left_inner_knuckle_joint: type revolute, parent xarm_gripper_base_link, child left_inner_knuckle, origin xyz=0 0.02 0.074098 rpy=0 0 0, axis 1 0 0, limit lower=0 upper=0.85 effort=50 velocity=2, mimic joint=drive_joint multiplier=1 offset=0
- added joint right_finger_joint: type revolute, parent right_outer_knuckle, child right_finger, origin xyz=0 -0.035465 0.042039 rpy=0 0 0, axis 1 0 0, limit lower=0 upper=0.85 effort=50 velocity=2, mimic joint=drive_joint multiplier=1 offset=0
- added joint right_inner_knuckle_joint: type revolute, parent xarm_gripper_base_link, child right_inner_knuckle, origin xyz=0 -0.02 0.074098 rpy=0 0 0, axis -1 0 0, limit lower=0 upper=0.85 effort=50 velocity=2, mimic joint=drive_joint multiplier=1 offset=0
- added joint right_outer_knuckle_joint: type revolute, parent xarm_gripper_base_link, child right_outer_knuckle, origin xyz=0 -0.035 0.059098 rpy=0 0 0, axis -1 0 0, limit lower=0 upper=0.85 effort=50 velocity=2, mimic joint=drive_joint multiplier=1 offset=0
